File: pcb/SoilMetrics-Lite.kicad_sch (KiCad schematic)
At the start: 23 parts, among them J1 USB_C_Receptacle_USB2.0_16P, J2 Conn_01x04, J3 Conn_02x03_Odd_Even, SW1 SW_Push, U1 MAX485E, U2 CH340C, U3 ATmega328P-P, Y1 16MHz

Commit message: added gerber and bom
Parts:
- D1: value LED -> Red; Link (none) -> https://robu.in/product/3mm-red-dip-led-pack-of-50/; Price (none) -> 1.51
- D2: value LED -> yellow; Link (none) -> https://robu.in/product/3-mm-dip-led-yellow-50-pcs/; Price (none) -> 1
- D3: value LED -> green; Link (none) -> https://robu.in/product/3mm-green-dip-led-pack-of-50/; Price (none) -> 1.35
- J3: Link (none) -> https://robu.in/product/ds1021-2x3sf11-b-connfly-2x3-pin-2-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; Price (none) -> 3.44
- R4: Link (none) -> https://robu.in/product/1k-ohm-1-4w-0805-surface-mount-chip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; Price (none) -> 0.54
- U1: Link (none) -> https://robu.in/product/max485edtr-xblw-sop-8-rs-485-rs-422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; Price (none) -> 24
- U2: Link (none) -> https://techiesms.com/product/ch340c-usb-to-serial-converte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; Price (none) -> 45
- U3: Link (none) -> https://robu.in/product/atmega328p-pu-pdip-28-microcontroll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; Price (none) -> 339; S-price (none) -> 6; Socket (none) -> https://robu.in/product/28-pin-narrow-dip-ic-socket-base-ad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
